Commit message: ピックプレイスデモ完成

File: urdf/model.urdf (robot description, URDF)
Before this commit: robot firefighter, 6 links, 5 joints
Links:
- link base: mass 1 -> 0.1; geometry visual mesh filename=daes/base.STL
- link base_rot: mass 1 -> 0.1; geometry visual mesh filename=daes/base_rot.obj
- link link_1: mass 1 -> 0.1; geometry visual mesh filename=daes/link_1.obj
- link link_2: mass 1 -> 0.1; geometry visual mesh filename=daes/link_2.obj
- link link_3: mass 1 -> 0.1; geometry visual mesh filename=daes/link_3_2.obj
- link link_end: mass 1 -> 0.1

Commit message: ピックプレイスなんとなく完成

File: urdf/model.urdf (robot description, URDF)
Before this commit: robot firefighter, 6 links, 5 joints
Links:
- link link_end: geometry visual mesh filename=daes/link_end_2.obj
